File: minidrone/minidrone.kicad_pcb (KiCad board)
At the start: 2 copper layers, 162.5 x 133.3 mm, 109 parts, among them J1 Conn_01x10, J2 OUT, J3 EXT GATE, J4 GATE, J5 GATE, Q1 BC337, Q2 BC337, Q3 BC337, Q4 BC337, Q5 BC337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

Commit message: Complete initial layout
Parts:
- added H21: MountingHole, MountingHole:MountingHole_3.2mm_M3, F.Cu at (67.3, 156.2)
- added H22: MountingHole, MountingHole:MountingHole_3.2mm_M3, F.Cu at (67.3, 29.2)
- added H23: MountingHole, MountingHole:MountingHole_3.2mm_M3, F.Cu at (125.7, 156.2)
- added H24: MountingHole, MountingHole:MountingHole_3.2mm_M3, F.Cu at (125.7, 29.2)
- SW7: footprint Button_Switch_Keyboard:SW_Cherry_MX_1.00u_PCB -> kosmo-lib:SW_Kailh_Choc_1.00u_PCB
- moved R21 121.4 mm to (201.9, 50.8)
- moved R22 112.9 mm to (204.5, 50.8), turned to 90 degrees
- moved R16 80.9 mm to (221.6, 54.0), turned to 180 degrees
- moved R25 79.4 mm to (194.3, 130.2), turned to 0 degrees
- moved R11 75.9 mm to (167.0, 36.2), turned to -90 degrees
- moved RV9 72.4 mm to (175.9, 132.1)
- moved R31 71.1 mm to (179.7, 129.5)
- moved R32 71.1 mm to (182.2, 132.1)
- moved JP1 71.1 mm to (184.8, 130.2), turned to -90 degrees
- moved R29 68.6 mm to (214.6, 125.1), turned to 0 degrees
- moved R27 66.8 mm to (204.5, 132.7), turned to 180 degrees
- moved D8 64.1 mm to (199.4, 87.6), turned to 0 degrees
- moved Q9 62.2 mm to (206.8, 130.2), turned to 0 degrees
- moved C6 61.2 mm to (167.0, 48.9), turned to -90 degrees
- moved D7 58.8 mm to (201.9, 67.3)
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Connections:
- net /CV renamed /PITCH
- net Net-(Q8-Pad1) renamed /VCA_DA_SIG
- net Net-(Q8-Pad2) renamed /VCA_IN
- net Net-(Q8-Pad3) renamed /VCA_CE
- net Net-(Q9-Pad1) renamed /VCA_DA_REF
- net Net-(R20-Pad2) renamed /VCA_CV
- net Net-(R29-Pad2) renamed /VCA_OUT
- U2 pad 1: /EG_OUT -> /EG_COMP_OUT
- U2 pad 2: /EG_OUT -> /EG_VTH
- U2 pad 3: /EG_CAP -> /EG_TRIG
- U2 pad 5: /EG_TRIG -> /EG_CAP
- U2 pad 6: /EG_VTH -> /EG_OUT
- U2 pad 7: /EG_COMP_OUT -> /EG_OUT
Routing:
- net +12V: track 93.8 -> 247.2 mm
- net -12V: track 141.3 -> 271.9 mm
- net /VCA_IN: track 0.00 -> 124.0 mm
- net Net-(C6-Pad1): track 0.00 -> 59.4 mm
- net /EG_TRIG: track 0.00 -> 45.6 mm
- net /VIN: track 113.2 -> 153.5 mm
- net /EG_CAP: track 0.00 -> 40.1 mm
- net /VCA_CV: track 5.08 -> 36.8 mm
- net /VCA_BIAS: track 6.35 -> 36.5 mm
- net Net-(D9-Pad1): track 0.00 -> 30.1 mm
- net /EG_OUT: track 0.02 -> 24.1 mm
- net /PITCH: track 0.00 -> 20.6 mm
- net /Oscillator Bank/OUT: track 76.9 -> 97.2 mm
- net Net-(D8-Pad2): track 0.00 -> 17.2 mm
- net Net-(D7-Pad1): track 0.00 -> 17.0 mm
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- added copper zone on B.Cu, net GND
Other:
- board text added: "MINIDRONE"

Commit message: Complete cosmetics layout
Parts:
- moved C12 2.54 mm to (194.3, 85.1)
- moved C13 2.54 mm to (207.0, 82.5)
- moved C3 2.54 mm to (181.5, 96.5)
- moved C4 2.54 mm to (181.6, 120.7)
- moved C5 2.54 mm to (181.6, 144.8)
- moved C7 2.54 mm to (207.0, 85.1)
- moved D7 2.54 mm to (199.4, 67.3)
- moved J4 2.54 mm to (205.1, 106.7)
- moved Q1 2.54 mm to (179.1, 54.0)
- moved Q2 2.54 mm to (179.1, 77.7)
- moved Q3 2.54 mm to (179.1, 101.0)
- moved Q4 2.54 mm to (179.1, 125.1)
- moved Q5 2.54 mm to (179.1, 137.2)
- moved R16 2.54 mm to (219.1, 54.0)
- moved R17 2.54 mm to (199.4, 90.2)
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Other:
- board size 162.5 x 133.3 mm -> 160 x 133.3 mm
- board text added: "JLCJLCJLCJLC"
- board text added: "M I N I D R O N E"
- board text added: "MINIDRONE Front Panel github.com/mprosk/minidrone Max Proskauer v0.1 May 2022"
- board text added: "github.com/mprosk/minidrone Max Proskauer v0.1 May 2022"
- board text removed: "MINIDRONE"
