File: minidrone/front_panel.kicad_sch (KiCad schematic)
At the start: 22 parts, among them J5 GATE, SW7 GATE

Commit message: Complete initial layout
Parts:
- added H21, H22, H23, H24: MountingHole, MountingHole:MountingHole_3.2mm_M3, symbol Mechanical:MountingHole
- SW7: footprint Button_Switch_Keyboard:SW_Cherry_MX_1.00u_PCB -> kosmo-lib:SW_Kailh_Choc_1.00u_PCB
Changed lines of the file:
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@@
+    )
+  )
+  (symbol (lib_id "Mechanical:MountingHole") (at 92.71 152.4 0) (unit 1)
+    (in_bom yes) (on_board yes) (fields_autoplaced)
+    (property "Reference" "H22" (id 0) (at 95.25 151.1299 0)
+      (effects (font (size 1.27 1.27)) (justify left))
+    )
+    (property "Value" "MountingHole" (id 1) (at 95.25 153.6699 0)
+      (effects (font (size 1.27 1.27)) (justify left))
+    )
+    (property "Footprint" "MountingHole:MountingHole_3.2mm_M3" (id 2) (at 92.71 152.4 0)
+      (effects (font (size 1.27 1.27)) hide)
+    )
+    (property "Datasheet" "~" (id 3) (at 92.71 152.4 0)
+      (effects (font (size 1.27 1.27)) hide)
+    )
+  )
+  (symbol (lib_id "Mechanical:MountingHole") (at 92.71 158.75 0) (unit 1)
+    (in_bom yes) (on_board yes) (fields_autoplaced)
+    (property "Reference" "H23" (id 0) (at 95.25 157.4799 0)
+      (effects (font (size 1.27 1.27)) (justify left))
+    )
+    (property "Value" "MountingHole" (id 1) (at 95.25 160.0199 0)
+      (effects (font (size 1.27 1.27)) (justify left))
+    )
+    (property "Footprint" "MountingHole:MountingHole_3.2mm_M3" (id 2) (at 92.71 158.75 0)
+      (effects (font (size 1.27 1.27)) hide)
+    )
+    (property "Datasheet" "~" (id 3) (at 92.71 158.75 0)
+      (effects (font (size 1.27 1.27)) hide)
     )
   )
@@
     )
     (property "Datasheet" "~" (id 3) (at 118.11 118.11 0)
+      (effects (font (size 1.27 1.27)) hide)
+    )
+  )
+  (symbol (lib_id "Mechanical:MountingHole") (at 92.71 165.1 0) (unit 1)
+    (in_bom yes) (on_board yes) (fields_autoplaced)
+    (property "Reference" "H24" (id 0) (at 95.25 163.8299 0)
+      (effects (font (size 1.27 1.27)) (justify left))
+    )
+    (property "Value" "MountingHole" (id 1) (at 95.25 166.3699 0)
+      (effects (font (size 1.27 1.27)) (justify left))
+    )
+    (property "Footprint" "MountingHole:MountingHole_3.2mm_M3" (id 2) (at 92.71 165.1 0)
+      (effects (font (size 1.27 1.27)) hide)
+    )
+    (property "Datasheet" "~" (id 3) (at 92.71 165.1 0)
+      (effects (font (size 1.27 1.27)) hide)
+    )
+  )
+  (symbol (lib_id "Mechanical:MountingHole") (at 92.71 146.05 0) (unit 1)
+    (in_bom yes) (on_board yes) (fields_autoplaced)
+    (property "Reference" "H21" (id 0) (at 95.25 144.7799 0)
+      (effects (font (size 1.27 1.27)) (justify left))
+    )
+    (property "Value" "MountingHole" (id 1) (at 95.25 147.3199 0)
+      (effects (font (size 1.27 1.27)) (justify left))
+    )
+    (property "Footprint" "MountingHole:MountingHole_3.2mm_M3" (id 2) (at 92.71 146.05 0)
+      (effects (font (size 1.27 1.27)) hide)
+    )
+    (property "Datasheet" "~" (id 3) (at 92.71 146.05 0)
       (effects (font (size 1.27 1.27)) hide)
     )
@@
     (property "Reference" "SW7" (id 0) (at 189.23 130.81 0))
     (property "Value" "GATE" (id 1) (at 189.23 133.35 0))
-    (property "Footprint" "Button_Switch_Keyboard:SW_Cherry_MX_1.00u_PCB" (id 2) (at 189.23 137.16 0)
-      (effects (font (size 1.27 1.27)) hide)
-    )
+    (property "Footprint" "kosmo-lib:SW_Kailh_Choc_1.00u_PCB" (id 2) (at 189.23 137.16 0)
+      (effects (font (size 1.27 1.27)) hide)
+    )

Commit message: Export schematic to PDF
Other:
- company: (none) -> Max Proskauer
- title: (none) -> Front Panel
Changed lines of the file:
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@@
 (kicad_sch (version 20211123) (generator eeschema)
-  (paper "A4")
+  (paper "USLetter")
+  (title_block
+    (title "Front Panel")
+    (date "2022-05-27")
+    (rev "0.1")
+    (company "Max Proskauer")
+  )
   (wire (pts (xy 194.31 137.16) (xy 196.85 137.16))
     (stroke (width 0) (type default) (color 0 0 0 0))
