File: minidrone/osc_bank.kicad_sch (KiCad schematic)
At the start: 35 parts, among them Q1 BC337, Q2 BC337, Q3 BC337, Q4 BC337, Q5 BC337, SW1 SW_SPDT, SW2 SW_SPDT, SW3 SW_SPDT, SW4 SW_SPDT, SW5 SW_SPDT

Commit message: Correct pot footprints. continue layout
Parts:
- R10, R2, R4, R6, R8: footprint Resistor_THT:R_Axial_DIN0207_L6.3mm_D2.5mm_P10.16mm_Horizontal -> Resistor_THT:R_Axial_DIN0207_L6.3mm_D2.5mm_P2.54mm_Vertical
- RV1, RV2, RV3, RV4, RV5: footprint Potentiometer_THT:Potentiometer_Bourns_PTV09A-1_Single_Vertical -> minidrone:Bourns_PVT09A
Changed lines of the file:
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@@
       (effects (font (size 1.27 1.27)) (justify right))
     )
-    (property "Footprint" "Potentiometer_THT:Potentiometer_Bourns_PTV09A-1_Single_Vertical" (id 2) (at 135.89 92.71 0)
+    (property "Footprint" "minidrone:Bourns_PVT09A" (id 2) (at 135.89 92.71 0)
       (effects (font (size 1.27 1.27)) hide)
     )
@@
     (property "Reference" "R6" (id 0) (at 147.32 96.52 90))
     (property "Value" "100k" (id 1) (at 147.32 99.06 90))
-    (property "Footprint" "Resistor_THT:R_Axial_DIN0207_L6.3mm_D2.5mm_P10.16mm_Horizontal" (id 2) (at 147.32 99.822 90)
+    (property "Footprint" "Resistor_THT:R_Axial_DIN0207_L6.3mm_D2.5mm_P2.54mm_Vertical" (id 2) (at 147.32 99.822 90)
       (effects (font (size 1.27 1.27)) hide)
     )
@@
     (property "Reference" "R4" (id 0) (at 104.14 96.52 90))
     (property "Value" "100k" (id 1) (at 104.14 99.06 90))
-    (property "Footprint" "Resistor_THT:R_Axial_DIN0207_L6.3mm_D2.5mm_P10.16mm_Horizontal" (id 2) (at 104.14 99.822 90)
+    (property "Footprint" "Resistor_THT:R_Axial_DIN0207_L6.3mm_D2.5mm_P2.54mm_Vertical" (id 2) (at 104.14 99.822 90)
       (effects (font (size 1.27 1.27)) hide)
     )
@@
     (property "Reference" "R8" (id 0) (at 190.5 96.52 90))
     (property "Value" "100k" (id 1) (at 190.5 99.06 90))
-    (property "Footprint" "Resistor_THT:R_Axial_DIN0207_L6.3mm_D2.5mm_P10.16mm_Horizontal" (id 2) (at 190.5 99.822 90)
+    (property "Footprint" "Resistor_THT:R_Axial_DIN0207_L6.3mm_D2.5mm_P2.54mm_Vertical" (id 2) (at 190.5 99.822 90)
       (effects (font (size 1.27 1.27)) hide)
     )
@@
     (property "Reference" "R2" (id 0) (at 60.96 96.52 90))
     (property "Value" "100k" (id 1) (at 60.96 99.06 90))
-    (property "Footprint" "Resistor_THT:R_Axial_DIN0207_L6.3mm_D2.5mm_P10.16mm_Horizontal" (id 2) (at 60.96 99.822 90)
+    (property "Footprint" "Resistor_THT:R_Axial_DIN0207_L6.3mm_D2.5mm_P2.54mm_Vertical" (id 2) (at 60.96 99.822 90)
       (effects (font (size 1.27 1.27)) hide)
     )
@@
       (effects (font (size 1.27 1.27)) (justify right))
     )
-    (property "Footprint" "Potentiometer_THT:Potentiometer_Bourns_PTV09A-1_Single_Vertical" (id 2) (at 92.71 92.71 0)
+    (property "Footprint" "minidrone:Bourns_PVT09A" (id 2) (at 92.71 92.71 0)
       (effects (font (size 1.27 1.27)) hide)
     )
@@
       (effects (font (size 1.27 1.27)) (justify right))
     )
-    (property "Footprint" "Potentiometer_THT:Potentiometer_Bourns_PTV09A-1_Single_Vertical" (id 2) (at 49.53 92.71 0)
+    (property "Footprint" "minidrone:Bourns_PVT09A" (id 2) (at 49.53 92.71 0)
       (effects (font (size 1.27 1.27)) hide)
     )
@@
     (property "Reference" "R10" (id 0) (at 233.68 96.52 90))
     (property "Value" "100k" (id 1) (at 233.68 99.06 90))
-    (property "Footprint" "Resistor_THT:R_Axial_DIN0207_L6.3mm_D2.5mm_P10.16mm_Horizontal" (id 2) (at 233.68 99.822 90)
+    (property "Footprint" "Resistor_THT:R_Axial_DIN0207_L6.3mm_D2.5mm_P2.54mm_Vertical" (id 2) (at 233.68 99.822 90)
       (effects (font (size 1.27 1.27)) hide)
     )
@@
       (effects (font (size 1.27 1.27)) (justify right))
     )
-    (property "Footprint" "Potentiometer_THT:Potentiometer_Bourns_PTV09A-1_Single_Vertical" (id 2) (at 222.25 92.71 0)
+    (property "Footprint" "minidrone:Bourns_PVT09A" (id 2) (at 222.25 92.71 0)
       (effects (font (size 1.27 1.27)) hide)
     )
@@
       (effects (font (size 1.27 1.27)) (justify right))
     )
-    (property "Footprint" "Potentiometer_THT:Potentiometer_Bourns_PTV09A-1_Single_Vertical" (id 2) (at 179.07 92.71 0)
-      (effects (font (size 1.27 1.27)) hide)
-    )
+    (property "Footprint" "minidrone:Bourns_PVT09A" (id 2) (at 179.07 92.71 0)
+      (effects (font (size 1.27 1.27)) hide)
+    )

Commit message: Continue layout
Parts:
- R10, R2, R4, R6, R8: footprint Resistor_THT:R_Axial_DIN0207_L6.3mm_D2.5mm_P2.54mm_Vertical -> Resistor_THT:R_Axial_DIN0207_L6.3mm_D2.5mm_P10.16mm_Horizontal
Changed lines of the file:
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@@
     (property "Reference" "R6" (id 0) (at 147.32 96.52 90))
     (property "Value" "100k" (id 1) (at 147.32 99.06 90))
-    (property "Footprint" "Resistor_THT:R_Axial_DIN0207_L6.3mm_D2.5mm_P2.54mm_Vertical" (id 2) (at 147.32 99.822 90)
+    (property "Footprint" "Resistor_THT:R_Axial_DIN0207_L6.3mm_D2.5mm_P10.16mm_Horizontal" (id 2) (at 147.32 99.822 90)
       (effects (font (size 1.27 1.27)) hide)
     )
@@
     (property "Reference" "R4" (id 0) (at 104.14 96.52 90))
     (property "Value" "100k" (id 1) (at 104.14 99.06 90))
-    (property "Footprint" "Resistor_THT:R_Axial_DIN0207_L6.3mm_D2.5mm_P2.54mm_Vertical" (id 2) (at 104.14 99.822 90)
+    (property "Footprint" "Resistor_THT:R_Axial_DIN0207_L6.3mm_D2.5mm_P10.16mm_Horizontal" (id 2) (at 104.14 99.822 90)
       (effects (font (size 1.27 1.27)) hide)
     )
@@
     (property "Reference" "R8" (id 0) (at 190.5 96.52 90))
     (property "Value" "100k" (id 1) (at 190.5 99.06 90))
-    (property "Footprint" "Resistor_THT:R_Axial_DIN0207_L6.3mm_D2.5mm_P2.54mm_Vertical" (id 2) (at 190.5 99.822 90)
+    (property "Footprint" "Resistor_THT:R_Axial_DIN0207_L6.3mm_D2.5mm_P10.16mm_Horizontal" (id 2) (at 190.5 99.822 90)
       (effects (font (size 1.27 1.27)) hide)
     )
@@
     (property "Reference" "R2" (id 0) (at 60.96 96.52 90))
     (property "Value" "100k" (id 1) (at 60.96 99.06 90))
-    (property "Footprint" "Resistor_THT:R_Axial_DIN0207_L6.3mm_D2.5mm_P2.54mm_Vertical" (id 2) (at 60.96 99.822 90)
+    (property "Footprint" "Resistor_THT:R_Axial_DIN0207_L6.3mm_D2.5mm_P10.16mm_Horizontal" (id 2) (at 60.96 99.822 90)
       (effects (font (size 1.27 1.27)) hide)
     )
@@
     (property "Reference" "R10" (id 0) (at 233.68 96.52 90))
     (property "Value" "100k" (id 1) (at 233.68 99.06 90))
-    (property "Footprint" "Resistor_THT:R_Axial_DIN0207_L6.3mm_D2.5mm_P2.54mm_Vertical" (id 2) (at 233.68 99.822 90)
-      (effects (font (size 1.27 1.27)) hide)
-    )
+    (property "Footprint" "Resistor_THT:R_Axial_DIN0207_L6.3mm_D2.5mm_P10.16mm_Horizontal" (id 2) (at 233.68 99.822 90)
+      (effects (font (size 1.27 1.27)) hide)
+    )

Commit message: Lay out front panel. WIP updating mainboard layout
Parts:
- SW1, SW2, SW3, SW4, SW5: footprint modular:Switch_SPDT -> kosmo-lib:Switch_SPDT
- renumbered C5 to C1, C1 to C5
Connections:
- net at D1.2 (A), Q1.1 (C): now also C1.2; no longer C5.2
- net at Q1.2 (E), R2.2, RV1.1: now also C1.1; no longer C5.1
- net at Q5.2 (E), R10.2, RV5.1: now also C5.1; no longer C1.1
- net at D5.2 (A), Q5.1 (C): now also C5.2; no longer C1.2
Other:
- moved on the sheet: C1, C5
Changed lines of the file:
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@@
     (effects (font (size 1.27 1.27)) (justify left bottom))
   )
-  (text "High" (at 229.87 114.3 0)
+  (text "High" (at 57.15 114.3 0)
     (effects (font (size 1.27 1.27)) (justify left bottom))
   )
@@
     (effects (font (size 1.27 1.27)) (justify left bottom))
   )
-  (text "Low" (at 57.15 114.3 0)
+  (text "Low" (at 229.87 114.3 0)
     (effects (font (size 1.27 1.27)) (justify left bottom))
   )
@@
       (effects (font (size 1.27 1.27)) (justify right))
     )
-    (property "Footprint" "modular:Switch_SPDT" (id 2) (at 133.35 66.04 0)
+    (property "Footprint" "kosmo-lib:Switch_SPDT" (id 2) (at 133.35 66.04 0)
       (effects (font (size 1.27 1.27)) hide)
     )
@@
       (effects (font (size 1.27 1.27)) (justify right))
     )
-    (property "Footprint" "modular:Switch_SPDT" (id 2) (at 176.53 66.04 0)
+    (property "Footprint" "kosmo-lib:Switch_SPDT" (id 2) (at 176.53 66.04 0)
       (effects (font (size 1.27 1.27)) hide)
     )
@@
       (effects (font (size 1.27 1.27)) (justify right))
     )
-    (property "Footprint" "modular:Switch_SPDT" (id 2) (at 46.99 66.04 0)
+    (property "Footprint" "kosmo-lib:Switch_SPDT" (id 2) (at 46.99 66.04 0)
       (effects (font (size 1.27 1.27)) hide)
     )
@@
       (effects (font (size 1.27 1.27)) (justify right))
     )
-    (property "Footprint" "modular:Switch_SPDT" (id 2) (at 219.71 66.04 0)
+    (property "Footprint" "kosmo-lib:Switch_SPDT" (id 2) (at 219.71 66.04 0)
       (effects (font (size 1.27 1.27)) hide)
     )
@@
     (pin "2")
   )
-  (symbol (lib_id "Device:CP") (at 54.61 109.22 0) (unit 1)
-    (in_bom yes) (on_board yes)
-    (property "Reference" "C1" (id 0) (at 57.6072 108.0516 0)
-      (effects (font (size 1.27 1.27)) (justify left))
-    )
-    (property "Value" "10uF" (id 1) (at 57.6072 110.363 0)
-      (effects (font (size 1.27 1.27)) (justify left))
-    )
-    (property "Footprint" "Capacitor_THT:CP_Radial_D5.0mm_P2.50mm" (id 2) (at 55.5752 113.03 0)
-      (effects (font (size 1.27 1.27)) hide)
-    )
-    (property "Datasheet" "~" (id 3) (at 54.61 109.22 0)
+  (symbol (lib_id "Device:CP") (at 227.33 109.22 0) (unit 1)
+    (in_bom yes) (on_board yes)
+    (property "Reference" "C5" (id 0) (at 230.3272 108.0516 0)
+      (effects (font (size 1.27 1.27)) (justify left))
+    )
+    (property "Value" "10uF" (id 1) (at 230.3272 110.363 0)
+      (effects (font (size 1.27 1.27)) (justify left))
+    )
+    (property "Footprint" "Capacitor_THT:CP_Radial_D5.0mm_P2.50mm" (id 2) (at 228.2952 113.03 0)
+      (effects (font (size 1.27 1.27)) hide)
+    )
+    (property "Datasheet" "~" (id 3) (at 227.33 109.22 0)
       (effects (font (size 1.27 1.27)) hide)
     )
@@
       (effects (font (size 1.27 1.27)) (justify right))
     )
-    (property "Footprint" "modular:Switch_SPDT" (id 2) (at 90.17 66.04 0)
+    (property "Footprint" "kosmo-lib:Switch_SPDT" (id 2) (at 90.17 66.04 0)
       (effects (font (size 1.27 1.27)) hide)
     )
@@
     (pin "2")
   )
-  (symbol (lib_id "Device:CP") (at 227.33 109.22 0) (unit 1)
-    (in_bom yes) (on_board yes)
-    (property "Reference" "C5" (id 0) (at 230.3272 108.0516 0)
-      (effects (font (size 1.27 1.27)) (justify left))
-    )
-    (property "Value" "1uF" (id 1) (at 230.3272 110.363 0)
-      (effects (font (size 1.27 1.27)) (justify left))
-    )
-    (property "Footprint" "Capacitor_THT:CP_Radial_D5.0mm_P2.50mm" (id 2) (at 228.2952 113.03 0)
-      (effects (font (size 1.27 1.27)) hide)
-    )
-    (property "Datasheet" "~" (id 3) (at 227.33 109.22 0)
-      (effects (font (size 1.27 1.27)) hide)
-    )
+  (symbol (lib_id "Device:CP") (at 54.61 109.22 0) (unit 1)
+    (in_bom yes) (on_board yes)
+    (property "Reference" "C1" (id 0) (at 57.6072 108.0516 0)
+      (effects (font (size 1.27 1.27)) (justify left))
+    )
+    (property "Value" "1uF" (id 1) (at 57.6072 110.363 0)
+      (effects (font (size 1.27 1.27)) (justify left))
+    )
+    (property "Footprint" "Capacitor_THT:CP_Radial_D5.0mm_P2.50mm" (id 2) (at 55.5752 113.03 0)
+      (effects (font (size 1.27 1.27)) hide)
+    )
+    (property "Datasheet" "~" (id 3) (at 54.61 109.22 0)
+      (effects (font (size 1.27 1.27)) hide)
+    )

Commit message: Fix schematic issues identified in first production run. PCB fixes TODO!
Connections:
- net at R7.1, RV4.2: now also RV4.1; no longer RV4.3
- net at C3.1, Q3.2 (E), R6.2: now also RV3.3; no longer RV3.1
- net at R5.1, RV3.2: now also RV3.1; no longer RV3.3
- net at C1.1, Q1.2 (E), R2.2: now also RV1.3; no longer RV1.1
- net at C2.1, Q2.2 (E), R4.2: now also RV2.3; no longer RV2.1
- net at C4.1, Q4.2 (E), R8.2: now also RV4.3; no longer RV4.1
- net at R9.1, RV5.2: now also RV5.1; no longer RV5.3
- net at C5.1, Q5.2 (E), R10.2: now also RV5.3; no longer RV5.1
- net at R3.1, RV2.2: now also RV2.1; no longer RV2.3
- net at R1.1, RV1.2: now also RV1.1; no longer RV1.3
Changed lines of the file:
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@@
     (pin "2")
   )
-  (symbol (lib_id "Device:R_POT") (at 135.89 92.71 0) (mirror x) (unit 1)
-    (in_bom yes) (on_board yes)
-    (property "Reference" "RV3" (id 0) (at 134.1374 93.8784 0)
-      (effects (font (size 1.27 1.27)) (justify right))
-    )
-    (property "Value" "10k" (id 1) (at 134.1374 91.567 0)
+  (symbol (lib_id "Device:R_POT") (at 135.89 92.71 0) (unit 1)
+    (in_bom yes) (on_board yes)
+    (property "Reference" "RV3" (id 0) (at 134.1374 91.5416 0)
+      (effects (font (size 1.27 1.27)) (justify right))
+    )
+    (property "Value" "10k" (id 1) (at 134.1374 93.853 0)
       (effects (font (size 1.27 1.27)) (justify right))
     )
@@
     (pin "2")
   )
-  (symbol (lib_id "Device:R_POT") (at 92.71 92.71 0) (mirror x) (unit 1)
-    (in_bom yes) (on_board yes)
-    (property "Reference" "RV2" (id 0) (at 90.9574 93.8784 0)
-      (effects (font (size 1.27 1.27)) (justify right))
-    )
-    (property "Value" "10k" (id 1) (at 90.9574 91.567 0)
+  (symbol (lib_id "Device:R_POT") (at 92.71 92.71 0) (unit 1)
+    (in_bom yes) (on_board yes)
+    (property "Reference" "RV2" (id 0) (at 90.9574 91.5416 0)
+      (effects (font (size 1.27 1.27)) (justify right))
+    )
+    (property "Value" "10k" (id 1) (at 90.9574 93.853 0)
       (effects (font (size 1.27 1.27)) (justify right))
     )
@@
     (pin "2")
   )
-  (symbol (lib_id "Device:R_POT") (at 49.53 92.71 0) (mirror x) (unit 1)
-    (in_bom yes) (on_board yes)
-    (property "Reference" "RV1" (id 0) (at 47.7774 93.8784 0)
-      (effects (font (size 1.27 1.27)) (justify right))
-    )
-    (property "Value" "10k" (id 1) (at 47.7774 91.567 0)
+  (symbol (lib_id "Device:R_POT") (at 49.53 92.71 0) (unit 1)
+    (in_bom yes) (on_board yes)
+    (property "Reference" "RV1" (id 0) (at 47.7774 91.5416 0)
+      (effects (font (size 1.27 1.27)) (justify right))
+    )
+    (property "Value" "10k" (id 1) (at 47.7774 93.853 0)
       (effects (font (size 1.27 1.27)) (justify right))
     )
@@
     (pin "1")
   )
-  (symbol (lib_id "Device:R_POT") (at 222.25 92.71 0) (mirror x) (unit 1)
-    (in_bom yes) (on_board yes)
-    (property "Reference" "RV5" (id 0) (at 220.4974 93.8784 0)
-      (effects (font (size 1.27 1.27)) (justify right))
-    )
-    (property "Value" "10k" (id 1) (at 220.4974 91.567 0)
+  (symbol (lib_id "Device:R_POT") (at 222.25 92.71 0) (unit 1)
+    (in_bom yes) (on_board yes)
+    (property "Reference" "RV5" (id 0) (at 220.4974 91.5416 0)
+      (effects (font (size 1.27 1.27)) (justify right))
+    )
+    (property "Value" "10k" (id 1) (at 220.4974 93.853 0)
       (effects (font (size 1.27 1.27)) (justify right))
     )
@@
     (pin "2")
   )
-  (symbol (lib_id "Device:R_POT") (at 179.07 92.71 0) (mirror x) (unit 1)
-    (in_bom yes) (on_board yes)
-    (property "Reference" "RV4" (id 0) (at 177.3174 93.8784 0)
-      (effects (font (size 1.27 1.27)) (justify right))
-    )
-    (property "Value" "10k" (id 1) (at 177.3174 91.567 0)
-      (effects (font (size 1.27 1.27)) (justify right))
-    )
+  (symbol (lib_id "Device:R_POT") (at 179.07 92.71 0) (unit 1)
+    (in_bom yes) (on_board yes)
+    (property "Reference" "RV4" (id 0) (at 177.3174 91.5416 0)
+      (effects (font (size 1.27 1.27)) (justify right))
+    )
+    (property "Value" "10k" (id 1) (at 177.3174 93.853 0)
+      (effects (font (size 1.27 1.27)) (justify right))
+    )
